File: z80handheld/z80handheld.kicad_pcb (KiCad board)
At the start: 2 copper layers, 137 parts, among them IC1 DS12885+, J1 Power, J2 Esp32 C3 Supermini Right, J3 SPI Screen, J4 Esp32 C3 Supermini Left, SW1 SW_Push_45deg, SW10 SW_Push_45deg, SW11 SW_Push_45deg, SW12 SW_Push_45deg, SW13 SW_Push_45deg, SW14 SW_Push_45deg, SW15 SW_Push_45deg, SW16 SW_Push_45deg, SW17 SW_Push_45deg, SW18 SW_Push_45deg, SW19 SW_Push_45deg, SW2 SW_Push_45deg, SW20 SW_Push_45deg, SW21 SW_Push_45deg, SW22 SW_Push_45deg, SW23 SW_Push_45deg, SW24 SW_Push_45deg, SW25 SW_Push_45deg, SW26 SW_Push_45deg, SW27 SW_Push_45deg, SW28 SW_Push_45deg, SW29 SW_Push_45deg, SW3 SW_Push_45deg, SW30 SW_Push_45deg, SW31 SW_Push_45deg, SW32 SW_Push_45deg, SW33 SW_Push_45deg, SW34 SW_Push_45deg, SW35 SW_Push_45deg, SW36 SW_Push_45deg, SW37 SW_Push_45deg, SW38 SW_Push_45deg, SW39 SW_Push_45deg, SW4 SW_Push_45deg, SW40 SW_Push_45deg, SW41 SW_Push_45deg, SW42 SW_Push_45deg, SW43 SW_Push_45deg, SW44 SW_Push_45deg, SW45 SW_Push_45deg, SW46 SW_Push_45deg, SW47 SW_Push_45deg, SW48 SW_Push_45deg, SW49 SW_Push_45deg, SW5 SW_Push_45deg, SW50 SW_Push_45deg, SW51 SW_Push_45deg, SW52 SW_Push_45deg, SW53 SW_Push_45deg, SW54 SW_Push_45deg, SW55 SW_Push_45deg, SW56 SW_Push_45deg, SW57 SW_Push_45deg, SW58 SW_Push_45deg, SW59 SW_Push_45deg, SW6 SW_Push_45deg, SW60 SW_Push_45deg, SW61 SW_Push_45deg, SW62 SW_Push_45deg, SW63 SW_Push_45deg, SW64 SW_Push_45deg, SW65 SW_Push, SW7 SW_Push_45deg, SW8 SW_Push_45deg, SW9 SW_Push_45deg, U1 74HC04, U10 Z84C00xxP, U11 74LS573 IO1, U12 HDSP-7501, U13 74LS573, U14 HDSP-7501, U15 74LS573, U16 16550 IO2, U17 16550 IO3, U2 4068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

Commit message: Add files via upload
Parts:
- BT1, BZ1: moved to B.Cu
- U8: value 28C256 -> 28C256 Additional
- moved U6 242.0 mm to (286.6, 177.4), turned to 180 degrees
- moved U5 237.3 mm to (271.0, 177.5), turned to 180 degrees
- moved U13 231.0 mm to (296.8, 177.3), turned to 180 degrees
- moved U15 230.3 mm to (306.9, 177.3), turned to 180 degrees
- moved U8 223.9 mm to (290.4, 139.3), turned to 90 degrees
- moved U10 211.8 mm to (265.2, 73.2)
- moved U16 211.8 mm to (246.8, 73.2)
- moved U17 211.8 mm to (228.4, 73.2)
- moved U9 211.8 mm to (281.7, 82.8)
- moved J1 195.8 mm to (283.5, 192.6), turned to 90 degrees
- moved U11 193.6 mm to (253.2, 154.6)
- moved U7 191.5 mm to (303.1, 82.7)
- moved Y1 189.5 mm to (232.3, 173.3), turned to 90 degrees
- moved U14 180.1 mm to (303.2, 187.2), turned to 90 degrees
- moved SW65 176.5 mm to (253.0, 193.0), turned to 180 degrees
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Connections:
- D12 pad 1: GND -> !WR
- D12 pad 2: !IORQ -> 5V
- D15 pad 1: GND -> !RD
- D15 pad 2: !RD -> 5V
- D18 pad 1: GND -> !IORQ
- D18 pad 2: !WR -> 5V
- D21 pad 1: GND -> !MREQ
- D21 pad 2: !INT -> 5V
- D24 pad 1: GND -> !M1
- D24 pad 2: !HALT -> 5V
- D6 pad 1: GND -> !HALT
- D6 pad 2: !M1 -> 5V
- D9 pad 1: GND -> !INT
- D9 pad 2: !MREQ -> 5V
- SW65 pad 1: 5V -> GND
- SW65 pad 2: GND -> !RESET
Routing:
- net GND: track 0.00 -> 560.1 mm, vias 0 -> 2
- net 5V: track 0.00 -> 558.3 mm, vias 0 -> 1
- net D2: track 0.00 -> 300.1 mm, vias 0 -> 2
- net D1: track 0.00 -> 251.3 mm, vias 0 -> 1
- net D0: track 0.00 -> 245.8 mm, vias 0 -> 3
- net D3: track 0.00 -> 241.7 mm, vias 0 -> 2
- net A7: track 0.00 -> 232.3 mm, vias 0 -> 3
- net D6: track 0.00 -> 224.5 mm, vias 0 -> 2
- net A0: track 0.00 -> 223.1 mm, vias 0 -> 3
- net D4: track 0.00 -> 221.2 mm, vias 0 -> 2
- net !WR: track 0.00 -> 219.9 mm, vias 0 -> 2
- net A5: track 0.00 -> 214.8 mm, vias 0 -> 2
- net A6: track 0.00 -> 214.6 mm, vias 0 -> 3
- net D5: track 0.00 -> 214.2 mm, vias 0 -> 2
- net A4: track 0.00 -> 210.4 mm, vias 0 -> 3
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Other:
- board outline added: 102.2 x 147.6 mm
- copper layers 2 -> 4
- board text added: "!BANK_0 !BANK_1 SIGNALS"
- board text added: "ADDRESS"
- board text added: "DATA"
- board text added: "M1 MREQ IORQ RD WR INT HALT"

Commit message: Add files via upload
Parts:
- added J5: Conn_01x40, Connector_PinHeader_2.54mm:PinHeader_1x40_P2.54mm_Vertical, F.Cu at (208.4, 70.1)
- added U18: 74AHCT1G32, Package_TO_SOT_SMD:SC-74A-5_1.55x2.9mm_P0.95mm, F.Cu at (305.2, 127.9)
- added U19: 74AHCT1G32, Package_TO_SOT_SMD:SC-74A-5_1.55x2.9mm_P0.95mm, F.Cu at (305.2, 133.1)
Connections:
- net Net-(U10-CLK) renamed CLK
- D3 pad 2: !MREQ -> BANK_0
- D31 pad 2: !MREQ -> A15
- U1 pad 12: !MREQ -> Net-(U7-~{CS})
- U1 pad 13: !MREQ -> A15
- U1 pad 3: !MREQ -> A15
- U10 pad 5: !MREQ -> A15
- U2 pad 2: !MREQ -> A15
- U3 pad 8: unconnected-(U3-Pad8) -> IO8
- U3 pad 9: unconnected-(U3-Pad9) -> IO1
- U6 pad 19: !MREQ -> BANK_0
- U7 pad 20: !MREQ -> Net-(U7-~{CS})
- U9 pad 20: !MREQ -> Net-(U9-~{CS})
Routing:
- net D2: track 300.1 -> 51.4 mm, vias 2 -> 0
- net A7: track 232.3 -> 0.00 mm, vias 3 -> 0
- net D6: track 224.5 -> 0.00 mm, vias 2 -> 0
- net A0: track 223.1 -> 0.00 mm, vias 3 -> 0
- net !WR: track 219.9 -> 0.00 mm, vias 2 -> 0
- net A5: track 214.8 -> 0.00 mm, vias 2 -> 0
- net A6: track 214.6 -> 0.00 mm, vias 3 -> 0
- net D5: track 214.2 -> 0.00 mm, vias 2 -> 0
- net A4: track 210.4 -> 0.00 mm, vias 3 -> 0
- net !MREQ: track 210.3 -> 0.00 mm, vias 5 -> 0
- net !RD: track 207.7 -> 0.00 mm, vias 2 -> 0
- net D7: track 206.2 -> 0.00 mm, vias 1 -> 0
- net D1: track 251.3 -> 47.8 mm, vias 1 -> 0
- net GND: track 560.1 -> 763.2 mm, vias 2 -> 0
- net D0: track 245.8 -> 44.2 mm, vias 3 -> 0
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Other:
- board size 102.2 x 147.6 mm -> 104 x 148.2 mm

Commit message: Add files via upload
Routing:
- net D5: track 0.00 -> 312.4 mm, vias 0 -> 4
- net D6: track 0.00 -> 281.5 mm, vias 0 -> 6
- net D7: track 0.00 -> 267.6 mm, vias 0 -> 7
- net D2: track 51.4 -> 316.9 mm, vias 0 -> 5
- net !RD: track 0.00 -> 264.5 mm, vias 0 -> 5
- net D0: track 44.2 -> 307.5 mm, vias 0 -> 7
- net !WR: track 0.00 -> 262.3 mm, vias 0 -> 6
- net !MREQ: track 0.00 -> 258.0 mm, vias 0 -> 7
- net A5: track 0.00 -> 256.1 mm, vias 0 -> 9
- net D1: track 47.8 -> 300.3 mm, vias 0 -> 7
- net !INT: track 0.00 -> 251.8 mm, vias 0 -> 5
- net A0: track 0.00 -> 250.3 mm, vias 0 -> 6
- net A6: track 0.00 -> 248.5 mm, vias 0 -> 6
- net D3: track 55.0 -> 298.2 mm, vias 0 -> 9
- net A4: track 0.00 -> 242.9 mm, vias 0 -> 6
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Other:
- board size 104 x 148.2 mm -> 104.7 x 148.2 mm
- copper layers 4 -> 2

Commit message: Add files via upload
Connections:
- U3 pad 10: Net-(U16-INTR) -> !INT
- U3 pad 11: !INT -> Net-(U16-INTR)
Routing:
- net GND: track 569.5 -> 637.4 mm, vias 16 -> 15
- net Net-(J2-Pin_8): track 122.1 -> 87.8 mm
- net Net-(U11-D3): track 85.5 -> 118.0 mm
- net IO1: track 218.2 -> 188.1 mm
- net Net-(U5-Q6): track 174.4 -> 147.2 mm, vias 12 -> 8
- net A12: track 194.2 -> 167.5 mm, vias 3 -> 5
- net Net-(U5-Q2): track 159.1 -> 134.1 mm, vias 10 -> 9
- net 5V: track 564.9 -> 585.5 mm, vias 12 -> 14
- net D2: track 316.9 -> 297.4 mm, vias 5 -> 9
- net !RESET: track 229.4 -> 210.0 mm, vias 4 -> 2
- net TX1: track 118.3 -> 136.2 mm, vias 1 -> 0
- net Net-(U11-D2): track 95.1 -> 112.1 mm
- net Net-(U7-~{CS}): track 115.9 -> 132.9 mm
- net D7: track 267.6 -> 284.4 mm, vias 7 -> 8
- net D5: track 312.4 -> 295.9 mm, vias 4 -> 7
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Other:
- board size 104.7 x 148.2 mm -> 105.2 x 148.2 mm

Commit message: Add files via upload
Parts:
- removed U19: 74AHCT1G32, Package_TO_SOT_SMD:SC-74A-5_1.55x2.9mm_P0.95mm
- U18: value 74AHCT1G32 -> 74HCT00; footprint Package_TO_SOT_SMD:SC-74A-5_1.55x2.9mm_P0.95mm -> Package_DIP:DIP-14_W7.62mm
- moved U18 96.6 mm to (209.8, 142.7), turned to 90 degrees
- moved BT1 47.9 mm to (257.9, 193.2), turned to -90 degrees
- moved Y2 33.1 mm to (243.1, 153.1), turned to 90 degrees
- moved Y1 11.8 mm to (234.3, 185.0), turned to 0 degrees
- moved IC1 8.89 mm to (235.7, 162.7), turned to -90 degrees
- moved Y3 4.95 mm to (216.3, 168.7)
- moved J2 4.55 mm to (226.0, 189.6)
- moved J4 4.55 mm to (208.2, 174.4)
- moved R2 4.55 mm to (225.0, 178.1)
- moved R3 4.55 mm to (220.9, 178.1)
- moved R5 4.55 mm to (212.8, 178.1)
- moved R1 4.55 mm to (229.1, 178.1)
- moved R4 4.55 mm to (216.9, 178.1)
- moved R6 4.55 mm to (208.8, 178.1)
- moved BZ1 4.39 mm to (233.3, 193.2)
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Connections:
- net A0 renamed /A0
- net A1 renamed /A1
- net A10 renamed /A10
- net A11 renamed /A11
- net A12 renamed /A12
- net A13 renamed /A13
- net A14 renamed /A14
- net A2 renamed /A2
- net A3 renamed /A3
- net A4 renamed /A4
- net A5 renamed /A5
- net A6 renamed /A6
- net A7 renamed /A7
- net A8 renamed /A8
- net A9 renamed /A9
- net D0 renamed /D0
- net D1 renamed /D1
- net D2 renamed /D2
- net D3 renamed /D3
- net D4 renamed /D4
- net D5 renamed /D5
- net D6 renamed /D6
- net D7 renamed /D7
- D3 pad 2: BANK_0 -> !CS_EEPROM
- D5 pad 2: !MREQ -> !CS_RAM
- U1 pad 12: Net-(U7-~{CS}) -> Net-(U1-Pad12)
- U1 pad 3: A15 -> !MREQ
- U1 pad 4: !MREQ -> Net-(U1-Pad4)
- U18 pad 2: !MREQ -> Net-(U1-Pad4)
- U18 pad 3: GND -> !CS_EEPROM
- U18 pad 4: Net-(U9-~{CS}) -> A15
- U18 pad 5: 5V -> Net-(U1-Pad4)
- U6 pad 18: !MREQ -> !CS_RAM
- U6 pad 19: BANK_0 -> !CS_EEPROM
- U7 pad 20: Net-(U7-~{CS}) -> !CS_RAM
- U8 pad 20: !MREQ -> !CS_EEPROM
- U9 pad 20: Net-(U9-~{CS}) -> !CS_Main
Routing:
- net !CS_RAM: track 0.00 -> 188.5 mm, vias 0 -> 4
- net Net-(U7-~{CS}): track 132.9 -> 0.00 mm
- net !CS_EEPROM: track 0.00 -> 132.0 mm, vias 0 -> 3
- net /D4: track 273.5 -> 380.3 mm, vias 6 -> 8
- net !CS_Main: track 0.00 -> 79.7 mm, vias 0 -> 4
- net !MREQ: track 260.6 -> 185.0 mm, vias 5 -> 9
- net BANK_0: track 71.7 -> 0.00 mm, vias 4 -> 0
- net IO1: track 188.1 -> 255.0 mm, vias 2 -> 7
- net Net-(U12-C): track 15.8 -> 77.6 mm, vias 2 -> 1
- net Net-(U1-Pad4): track 0.00 -> 60.1 mm, vias 0 -> 6
- net Net-(U9-~{CS}): track 59.2 -> 0.00 mm
- net /A0: track 252.5 -> 310.9 mm, vias 8 -> 10
- net /A3: track 191.0 -> 247.0 mm, vias 6 -> 9
- net /D0: track 292.9 -> 342.2 mm, vias 7 -> 8
- net GND: track 637.4 -> 685.7 mm, vias 15 -> 22
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
Commit message: Add files via upload
Parts:
- moved U8 61.5 mm to (265.6, 83.0), turned to 180 degrees
- moved U16 60.5 mm to (307.3, 73.9)
- moved U17 59.9 mm to (288.2, 73.9)
- moved U9 56.6 mm to (225.2, 83.0)
- moved U7 56.4 mm to (246.7, 83.0)
- moved U10 55.1 mm to (255.3, 127.4), turned to -90 degrees
- moved J3 4.09 mm to (208.6, 84.5)
- moved U15 0.77 mm to (307.7, 177.3)
- moved U14 0.73 mm to (303.9, 187.2)
Routing:
- net GND: track 685.7 -> 97.3 mm, vias 22 -> 0
- net 5V: track 616.3 -> 133.1 mm, vias 16 -> 0
- net (no net): track 0.00 -> 384.7 mm
- net /D4: track 380.3 -> 87.6 mm, vias 8 -> 0
- net /D1: track 326.7 -> 54.1 mm, vias 8 -> 0
- net /D0: track 342.2 -> 70.1 mm, vias 8 -> 0
- net /D2: track 341.0 -> 78.6 mm, vias 8 -> 0
- net /A0: track 310.9 -> 50.1 mm, vias 10 -> 0
- net IO1: track 255.0 -> 0.00 mm, vias 7 -> 0
- net /D3: track 333.2 -> 82.7 mm, vias 19 -> 0
- net !WR: track 290.8 -> 42.1 mm, vias 4 -> 0
- net !INT: track 244.4 -> 0.00 mm, vias 2 -> 0
- net /D5: track 326.4 -> 93.2 mm, vias 11 -> 0
- net /A7: track 264.7 -> 42.6 mm, vias 5 -> 0
- net /A6: track 263.8 -> 42.1 mm, vias 8 -> 0
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
Commit message: Add files via upload
Parts:
- U2: footprint PCM_Package_DIP_AKL:DIP-14_W7.62mm -> Package_DIP:DIP-14_W7.62mm
- U4: footprint PCM_Package_DIP_AKL:DIP-24_W7.62mm -> Package_DIP:DIP-24_W7.62mm
- moved J5 111.5 mm to (307.0, 122.0), turned to -90 degrees
- moved Y3 33.5 mm to (249.1, 175.7), turned to 180 degrees
- moved Y1 24.0 mm to (216.3, 169.1), turned to 90 degrees
- moved U18 23.3 mm to (225.2, 125.3), turned to -90 degrees
- moved U3 22.7 mm to (230.0, 143.2)
- moved U1 22.5 mm to (225.1, 135.4)
- moved U16 4.20 mm to (308.0, 69.8)
- moved U17 4.20 mm to (288.9, 69.8)
- moved U7 4.04 mm to (246.0, 79.0)
- moved U8 4.04 mm to (266.3, 79.0)
- moved U9 4.04 mm to (225.8, 79.0)
- moved J3 4.04 mm to (209.3, 80.5)
- moved SW65 1.52 mm to (251.8, 193.2)
- moved U2 0.92 mm to (230.0, 133.0)
Connections:
- IC1 pad 13: IO1 -> IO7
- U1 pad 1: IO1 -> Net-(U4-~{S0})
- U1 pad 10: Net-(U4-~{E1}) -> PullIO
- U1 pad 5: IO1 -> Net-(U4-~{S2})
- U1 pad 9: IO1 -> Net-(U4-~{S3})
- U2 pad 13: IO1 -> PullIO
- U3 pad 1: IO1 -> Net-(U4-~{S4})
- U3 pad 3: IO1 -> Net-(U4-~{S5})
- U3 pad 5: IO1 -> Net-(U4-~{S6})
- U3 pad 9: IO1 -> Net-(U4-~{S8})
- U4 pad 1: IO1 -> Net-(U4-~{S0})
- U4 pad 10: IO1 -> unconnected-(U4-~{S9}-Pad10)
- U4 pad 11: IO1 -> unconnected-(U4-~{S10}-Pad11)
- U4 pad 13: IO1 -> unconnected-(U4-~{S11}-Pad13)
- U4 pad 14: IO1 -> unconnected-(U4-~{S12}-Pad14)
- U4 pad 15: IO1 -> unconnected-(U4-~{S13}-Pad15)
- U4 pad 16: IO1 -> unconnected-(U4-~{S14}-Pad16)
- U4 pad 17: IO1 -> unconnected-(U4-~{S15}-Pad17)
- U4 pad 19: Net-(U4-~{E1}) -> PullIO
- U4 pad 3: IO1 -> Net-(U4-~{S2})
- U4 pad 4: IO1 -> Net-(U4-~{S3})
- U4 pad 5: IO1 -> Net-(U4-~{S4})
- U4 pad 6: IO1 -> Net-(U4-~{S5})
- U4 pad 7: IO1 -> Net-(U4-~{S6})
- U4 pad 8: IO1 -> IO7
- U4 pad 9: IO1 -> Net-(U4-~{S8})
Routing:
- net (no net): track 384.7 -> 0.00 mm
- net TX1: track 0.00 -> 270.7 mm
- net RX1: track 0.00 -> 268.5 mm
- net GND: track 97.3 -> 318.1 mm
- net 5V: track 133.1 -> 312.3 mm
- net Net-(J2-Pin_8): track 0.00 -> 130.1 mm
- net CLK: track 0.00 -> 126.6 mm
- net Net-(J2-Pin_7): track 0.00 -> 122.9 mm
- net Net-(J2-Pin_5): track 0.00 -> 117.1 mm
- net Net-(U4-~{S0}): track 0.00 -> 112.8 mm
- net Net-(J2-Pin_4): track 0.00 -> 107.0 mm
- net Net-(J2-Pin_3): track 0.00 -> 104.5 mm
- net Net-(J3-Pin_6): track 0.00 -> 91.2 mm
- net /D1: track 54.1 -> 144.6 mm
- net Net-(U11-D3): track 0.00 -> 89.7 mm, vias 0 -> 8
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Other:
- board size 105.2 x 148.2 mm -> 107.9 x 151.1 mm
