File: z80handheld/z80handheld.kicad_sch (KiCad schematic)
At the start: 82 parts, among them J1 Conn_01x08_Socket, J2 Conn_01x08_Socket, SW1 SW_Push_45deg, SW10 SW_Push_45deg, SW11 SW_Push_45deg, SW12 SW_Push_45deg, SW13 SW_Push_45deg, SW14 SW_Push_45deg, SW15 SW_Push_45deg, SW16 SW_Push_45deg, SW17 SW_Push_45deg, SW18 SW_Push_45deg, SW19 SW_Push_45deg, SW2 SW_Push_45deg, SW20 SW_Push_45deg, SW21 SW_Push_45deg, SW22 SW_Push_45deg, SW23 SW_Push_45deg, SW24 SW_Push_45deg, SW25 SW_Push_45deg, SW26 SW_Push_45deg, SW27 SW_Push_45deg, SW28 SW_Push_45deg, SW29 SW_Push_45deg, SW3 SW_Push_45deg, SW30 SW_Push_45deg, SW31 SW_Push_45deg, SW32 SW_Push_45deg, SW33 SW_Push_45deg, SW34 SW_Push_45deg, SW35 SW_Push_45deg, SW36 SW_Push_45deg, SW37 SW_Push_45deg, SW38 SW_Push_45deg, SW39 SW_Push_45deg, SW4 SW_Push_45deg, SW40 SW_Push_45deg, SW41 SW_Push_45deg, SW42 SW_Push_45deg, SW43 SW_Push_45deg, SW44 SW_Push_45deg, SW45 SW_Push_45deg, SW46 SW_Push_45deg, SW47 SW_Push_45deg, SW48 SW_Push_45deg, SW49 SW_Push_45deg, SW5 SW_Push_45deg, SW50 SW_Push_45deg, SW51 SW_Push_45deg, SW52 SW_Push_45deg, SW53 SW_Push_45deg, SW54 SW_Push_45deg, SW55 SW_Push_45deg, SW56 SW_Push_45deg, SW57 SW_Push_45deg, SW58 SW_Push_45deg, SW59 SW_Push_45deg, SW6 SW_Push_45deg, SW60 SW_Push_45deg, SW61 SW_Push_45deg, SW62 SW_Push_45deg, SW63 SW_Push_45deg, SW64 SW_Push_45deg, SW65 SW_Push, SW7 SW_Push_45deg, SW8 SW_Push_45deg, SW9 SW_Push_45deg, U1 Z84C00xxP, U10 74HC04, U11 74HC04, U12 16550 IO3, U2 CY62256-70PC, U3 28C256, U4 28C256, U5 74LS573 IO0, U6 74LS573 IO1, U7 16550 IO2, U8 4068, U9 74154, Y1 20MHZ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

Commit message: Add files via upload
Parts:
- added BZ1: Buzzer, symbol Device:Buzzer
- added D1, D2, D3, D4, D5, D6: LED, symbol Device:LED
- added J3: Conn_01x14_Pin, symbol Connector:Conn_01x14_Pin
- added J4: Conn_01x02_Pin, symbol Connector:Conn_01x02_Pin
- added J5: Conn_01x27_Pin, symbol Connector:Conn_01x27_Pin
- added U13, U14, U15: 74LS573, symbol 74xx:74LS573
- added U16, U17: HDSP-7501, Display_7Segment:HDSP-A151, symbol Display_Character:HDSP-7501
Connections:
- net IO8 is gone; now on an unnamed net: U11.10
- net !RD: now also U2.22 (~{OE}), U3.22 (~{OE}), U4.22 (~{OE})
- net !WR: now also U2.27 (~{WE}), U3.27 (~{WE}), U4.27 (~{WE})
- net 5V: now also J1.1 (Pin_1), U12.36 (~{CTS}), U12.37 (~{DSR}), U12.38 (~{DCD}), U12.39 (~{RI}), U7.36 (~{CTS}), U7.37 (~{DSR}), U7.38 (~{DCD}), U7.39 (~{RI}), J3.14 (Pin_14), J4.1 (Pin_1), U15.20 (VCC)
- net D0: now also U15.2 (D0)
- net D1: now also U15.3 (D1)
- net D2: now also U15.4 (D2)
- net D3: now also U15.5 (D3)
- net D4: now also U15.6 (D4)
- net D5: now also U15.7 (D5)
- net D6: now also U15.8 (D6)
- net D7: now also U15.9 (D7)
- net GND: now also J1.2 (Pin_2), BZ1.2 (-), J3.13 (Pin_13), J4.2 (Pin_2), U15.1 (OE), U15.10 (GND)
- net IO1: now also U10.1, U10.5, U10.9, U11.1, U11.3, U11.5, U11.9, U6.1 (OE), U8.13 (J), U9.1 (~{S0}), U9.10 (~{S9}), U9.11 (~{S10}), U9.13 (~{S11}), U9.14 (~{S12}), U9.15 (~{S13}), U9.16 (~{S14}), U9.17 (~{S15}), U9.2 (~{S1}), U9.3 (~{S2}), U9.4 (~{S3}), U9.5 (~{S4}), U9.6 (~{S5}), U9.7 (~{S6}), U9.8 (~{S7}), U9.9 (~{S8}); no longer U10.13, U10.4
- net IO4: now also U15.11 (Load)
- net TX1: now reaches U7.10 (SIN)
- net TX1: now also J2.1 (Pin_1)
- net RX1: now reaches U7.11 (SOUT)
- net RX1: now also J2.2 (Pin_2)
- net at U7.15 (~{BAUDOUT}): now also U7.9 (RCLK)
- net at U7.30 (INTR): now also U12.30 (INTR)
- net at J2.5 (Pin_5): now also J3.6 (Pin_6)
- net at J2.8 (Pin_8): now also J3.9 (Pin_9)
- net at U10.12: no longer U6.1 (OE)
- net TX2: now reaches U12.10 (SIN)
- net RX2: now reaches U12.11 (SOUT)
- net at U12.15 (~{BAUDOUT}): now also U12.9 (RCLK)
- net !INT: now reaches U1.16 (~{INT})
- net !INT: now also U11.11
- net at J1.3 (Pin_3): now also J3.7 (Pin_7)
- net at J1.4 (Pin_4): now also J3.8 (Pin_8)
- net at J1.5 (Pin_5): now also J3.10 (Pin_10)
- net at J1.6 (Pin_6): now also BZ1.1 (+)
- net at J1.7 (Pin_7): now also J3.11 (Pin_11)
- net at J1.8 (Pin_8): now also J3.12 (Pin_12)
- new net: D6.2 (A), U15.12 (Q7)
- new net: D1.2 (A), U15.17 (Q2)
- new net: U14.19 (Q0), U17.10 (A)
- new net: U14.14 (Q5), U17.2 (F)
- new net: U14.13 (Q6), U17.3 (G)
- new net: U14.15 (Q4), U17.4 (E)
- new net: U14.16 (Q3), U17.5 (D)
- new net: U14.12 (Q7), U17.7 (DP)
- new net: U14.17 (Q2), U17.8 (C)
- new net: U14.18 (Q1), U17.9 (B)
- new net: U13.12 (Q7), U16.7 (DP)
- new net: U13.13 (Q6), U16.3 (G)
- new net: U13.14 (Q5), U16.2 (F)
- new net: U13.15 (Q4), U16.4 (E)
- new net: U13.16 (Q3), U16.5 (D)
- new net: U13.17 (Q2), U16.8 (C)
- new net: U13.18 (Q1), U16.9 (B)
- new net: U13.19 (Q0), U16.10 (A)
- new net: D5.2 (A), U15.13 (Q6)
- new net: D4.2 (A), U15.14 (Q5)
- new net: D3.2 (A), U15.15 (Q4)
- new net: D2.2 (A), U15.16 (Q3)
- now unconnected: U10.3
- no-connect marks 0 -> 14
Other:
- note added: "D0-7 A0-7 TXRX 5VGND IO M1 RD WR ALE RESET INT"
- note added: "FOR DUAL 7SEGMENTS"
- note added: "FOR EXTENSION"
- note added: "X X X X X MISO LED SCK MOSI DC/RS RESET CS GND VCC"

Commit message: Add files via upload
Parts:
- removed J5: Conn_01x27_Pin, symbol Connector:Conn_01x27_Pin
- removed unit 2 of U10
- removed unit 6 of U10
- removed unit 4 of U11
- added BT1: Battery_Cell, Battery:BatteryHolder_MYOUNG_BS-07-A1BJ001_CR2032, symbol Device:Battery_Cell
- added D1, D10, D12, D13, D15, D16, D18, D19, D2, D21, D22, D24, D25, D26, D27, D28, D29, D3, D30, D31, D32, D33, D34, D35, D36, D37, D38, D39, D4, D5, D6, D7, D9: LED, LED_SMD:LED_1206_3216Metric_Pad1.42x1.75mm_HandSolder, symbol Device:LED
- added IC1: DS12885+, DS12885:DIP1524W51P254L3175H508Q24N, symbol DS12885+:DS12885+
- added R1, R2, R3: 10k, Resistor_THT:R_Axial_DIN0207_L6.3mm_D2.5mm_P7.62mm_Horizontal, symbol PCM_Resistor_AKL:R_Generic
- added R4, R6: 1k, Resistor_THT:R_Axial_DIN0207_L6.3mm_D2.5mm_P7.62mm_Horizontal, symbol PCM_Resistor_AKL:R_Generic
- added unit 2 of U1
- added unit 6 of U1
- added unit 4 of U3
- added Y2: Crystal 32768Hz, Crystal:Crystal_C38-LF_D3.0mm_L8.0mm_Vertical, symbol Device:Crystal
- BZ1: footprint (none) -> Buzzer_Beeper:Buzzer_12x9.5RM7.6
- D11: renamed from D2; footprint (none) -> LED_SMD:LED_1206_3216Metric_Pad1.42x1.75mm_HandSolder
- D14: renamed from D3; footprint (none) -> LED_SMD:LED_1206_3216Metric_Pad1.42x1.75mm_HandSolder
- D17: renamed from D4; footprint (none) -> LED_SMD:LED_1206_3216Metric_Pad1.42x1.75mm_HandSolder
- D20: renamed from D5; footprint (none) -> LED_SMD:LED_1206_3216Metric_Pad1.42x1.75mm_HandSolder
- D23: renamed from D6; footprint (none) -> LED_SMD:LED_1206_3216Metric_Pad1.42x1.75mm_HandSolder
- D8: renamed from D1; footprint (none) -> LED_SMD:LED_1206_3216Metric_Pad1.42x1.75mm_HandSolder
- J1: renamed from J4; value Conn_01x02_Pin -> Power; footprint (none) -> Connector_PinHeader_2.54mm:PinHeader_1x02_P2.54mm_Vertical
- J2: renamed from J1; value Conn_01x08_Socket -> Esp32 C3 Supermini Right; footprint (none) -> Connector_PinHeader_2.54mm:PinHeader_1x08_P2.54mm_Vertical
- J3: value Conn_01x14_Pin -> SPI Screen; footprint (none) -> Connector_PinHeader_2.54mm:PinHeader_1x14_P2.54mm_Vertical
- J4: renamed from J2; value Conn_01x08_Socket -> Esp32 C3 Supermini Left; footprint (none) -> Connector_PinHeader_2.54mm:PinHeader_1x08_P2.54mm_Vertical
- R5: renamed from R1; footprint (none) -> Resistor_THT:R_Axial_DIN0207_L6.3mm_D2.5mm_P7.62mm_Horizontal
- SW1, SW10, SW11, SW12, SW13, SW14, SW15, SW16, SW17, SW2, SW3, SW32, SW33, SW4, SW5, SW56, SW57, SW58, SW59, SW6, SW60, SW61, SW62, SW63, SW64, SW7, SW8, SW9: footprint (none) -> Button_Switch_SMD:SW_SPST_PTS810
- SW18: renamed from SW19; footprint (none) -> Button_Switch_SMD:SW_SPST_PTS810
- SW19: renamed from SW21; footprint (none) -> Button_Switch_SMD:SW_SPST_PTS810
- SW20: renamed from SW23; footprint (none) -> Button_Switch_SMD:SW_SPST_PTS810
- SW21: renamed from SW25; footprint (none) -> Button_Switch_SMD:SW_SPST_PTS810
- SW22: renamed from SW27; footprint (none) -> Button_Switch_SMD:SW_SPST_PTS810
- SW23: renamed from SW29; footprint (none) -> Button_Switch_SMD:SW_SPST_PTS810
- SW24: renamed from SW31; footprint (none) -> Button_Switch_SMD:SW_SPST_PTS810
- SW25: renamed from SW18; footprint (none) -> Button_Switch_SMD:SW_SPST_PTS810
- SW26: renamed from SW20; footprint (none) -> Button_Switch_SMD:SW_SPST_PTS810
- SW27: renamed from SW22; footprint (none) -> Button_Switch_SMD:SW_SPST_PTS810
- SW28: renamed from SW24; footprint (none) -> Button_Switch_SMD:SW_SPST_PTS810
- SW29: renamed from SW26; footprint (none) -> Button_Switch_SMD:SW_SPST_PTS810
- SW30: renamed from SW28; footprint (none) -> Button_Switch_SMD:SW_SPST_PTS810
- SW31: renamed from SW30; footprint (none) -> Button_Switch_SMD:SW_SPST_PTS810
- SW34: renamed from SW36; footprint (none) -> Button_Switch_SMD:SW_SPST_PTS810
- SW35: renamed from SW39; footprint (none) -> Button_Switch_SMD:SW_SPST_PTS810
- SW36: renamed from SW42; footprint (none) -> Button_Switch_SMD:SW_SPST_PTS810
- SW37: renamed from SW45; footprint (none) -> Button_Switch_SMD:SW_SPST_PTS810
- SW38: renamed from SW48; footprint (none) -> Button_Switch_SMD:SW_SPST_PTS810
- SW39: renamed from SW51; footprint (none) -> Button_Switch_SMD:SW_SPST_PTS810
- SW40: renamed from SW54; footprint (none) -> Button_Switch_SMD:SW_SPST_PTS810
- SW41: renamed from SW34; footprint (none) -> Button_Switch_SMD:SW_SPST_PTS810
- SW42: renamed from SW37; footprint (none) -> Button_Switch_SMD:SW_SPST_PTS810
- SW43: renamed from SW40; footprint (none) -> Button_Switch_SMD:SW_SPST_PTS810
- SW44: renamed from SW43; footprint (none) -> Button_Switch_SMD:SW_SPST_PTS810
- SW45: renamed from SW46; footprint (none) -> Button_Switch_SMD:SW_SPST_PTS810
- SW46: renamed from SW49; footprint (none) -> Button_Switch_SMD:SW_SPST_PTS810
- SW47: renamed from SW52; footprint (none) -> Button_Switch_SMD:SW_SPST_PTS810
- SW48: renamed from SW55; footprint (none) -> Button_Switch_SMD:SW_SPST_PTS810
- SW49: renamed from SW35; footprint (none) -> Button_Switch_SMD:SW_SPST_PTS810
- SW50: renamed from SW38; footprint (none) -> Button_Switch_SMD:SW_SPST_PTS810
- SW51: renamed from SW41; footprint (none) -> Button_Switch_SMD:SW_SPST_PTS810
- SW52: renamed from SW44; footprint (none) -> Button_Switch_SMD:SW_SPST_PTS810
- SW53: renamed from SW47; footprint (none) -> Button_Switch_SMD:SW_SPST_PTS810
- SW54: renamed from SW50; footprint (none) -> Button_Switch_SMD:SW_SPST_PTS810
- SW55: renamed from SW53; footprint (none) -> Button_Switch_SMD:SW_SPST_PTS810
- SW65: footprint (none) -> Button_Switch_THT:SW_PUSH_6mm
- U1: renamed from U10; footprint (none) -> Package_DIP:DIP-14_W7.62mm
- U11: renamed from U6; footprint (none) -> Package_DIP:DIP-20_W7.62mm
- U12: renamed from U16; footprint Display_7Segment:HDSP-A151 -> Display_7Segment:KCSC02-106
- U13, U5: footprint (none) -> Package_DIP:DIP-20_W7.62mm
- U14: renamed from U17; footprint Display_7Segment:HDSP-A151 -> Display_7Segment:KCSC02-106
- U15: renamed from U14; footprint (none) -> Package_DIP:DIP-20_W7.62mm
- U2: renamed from U8; footprint (none) -> PCM_Package_DIP_AKL:DIP-14_W7.62mm
- U3: renamed from U11; footprint (none) -> Package_DIP:DIP-14_W7.62mm
- U4: renamed from U9; footprint (none) -> PCM_Package_DIP_AKL:DIP-24_W7.62mm
- U6: renamed from U15; footprint (none) -> Package_DIP:DIP-20_W7.62mm
- U7: renamed from U2; footprint Package_DIP:DIP-28_W15.24mm -> Socket:DIP_Socket-28_W6.9mm_W7.62mm_W10.16mm_W12.7mm_W13.5mm_3M_228-4817-00-0602J
- U8: renamed from U3; footprint (none) -> Socket:DIP_Socket-28_W6.9mm_W7.62mm_W10.16mm_W12.7mm_W13.5mm_3M_228-4817-00-0602J
- U9: renamed from U4; footprint (none) -> Socket:DIP_Socket-28_W6.9mm_W7.62mm_W10.16mm_W12.7mm_W13.5mm_3M_228-4817-00-0602J
- renumbered U1 to U10, U7 to U16, U12 to U17, Y2 to Y3
Connections:
- net A15 is gone; now on net !MREQ: U10.5 (A_{15}), U2.2 (A)
- net !INT: now also D21.2 (A), IC1.19 (~{IRQ})
- net !IORQ: now also U10.20 (~{IORQ}), D12.2 (A)
- net !M1: now also U10.27 (~{M1}), D6.2 (A)
- net !RD: now also D15.2 (A), IC1.17 (DS)
- net !RESET: now also IC1.18 (~{RESET})
- net !WR: now also D18.2 (A), IC1.15 (R/~{W})
- net 5V: now also U13.20 (VCC), U15.20 (VCC), IC1.21 (~{RCLR}), IC1.24 (VCC), R1.1, R2.1, R3.1
- net A0: now also D1.2 (A), IC1.14 (AS)
- net A1: now also D2.2 (A)
- net A10: now also D26.2 (A)
- net A11: now also D27.2 (A)
- net A12: now also D28.2 (A)
- net A13: now also D29.2 (A)
- net A14: now also D30.2 (A)
- net A2: now also D4.2 (A)
- net A3: now also D7.2 (A)
- net A4: now also D10.2 (A)
- net A5: now also D13.2 (A)
- net A6: now also D16.2 (A)
- net A7: now also D19.2 (A)
- net A8: now also D22.2 (A)
- net A9: now also D25.2 (A)
- net D0: now also U13.2 (D0), U15.2 (D0), D32.2 (A), IC1.4 (AD0)
- net D1: now also U13.3 (D1), U15.3 (D1), D33.2 (A), IC1.5 (AD1)
- net D2: now also U13.4 (D2), U15.4 (D2), D34.2 (A), IC1.6 (AD2)
- net D3: now also U13.5 (D3), U15.5 (D3), D35.2 (A), IC1.7 (AD3)
- net D4: now also U13.6 (D4), U15.6 (D4), D36.2 (A), IC1.8 (AD4)
- net D5: now also U13.7 (D5), U15.7 (D5), D37.2 (A), IC1.9 (AD5)
- net D6: now also U13.8 (D6), U15.8 (D6), D38.2 (A), IC1.10 (AD6)
- net D7: now also U13.9 (D7), U15.9 (D7), D39.2 (A), IC1.11 (AD7)
- net GND: now also D11.1 (K), D14.1 (K), D17.1 (K), D20.1 (K), D23.1 (K), D8.1 (K), U13.1 (OE), U13.10 (GND), U15.1 (OE), U15.10 (GND), BT1.2 (-), D1.1 (K), D10.1 (K), D12.1 (K), D13.1 (K), D15.1 (K), D16.1 (K), D18.1 (K), D19.1 (K), D2.1 (K), D21.1 (K), D22.1 (K), D24.1 (K), D25.1 (K), D26.1 (K), D27.1 (K), D28.1 (K), D29.1 (K), D3.1 (K), D30.1 (K), D31.1 (K), D32.1 (K), D33.1 (K), D34.1 (K), D35.1 (K), D36.1 (K), D37.1 (K), D38.1 (K), D39.1 (K), D4.1 (K), D5.1 (K), D6.1 (K), D7.1 (K), D9.1 (K), IC1.1 (MOT), IC1.12 (GND_1), IC1.16 (GND_2), R4.1, R6.1
- net IO1: now also IC1.13 (~{CS})
- net IO5: now also U13.11 (Load)
- net IO6: now also U15.11 (Load)
- net at U14.1 (CA): now also U14.6 (CA), R6.2
- net !MREQ: now reaches U9.20 (~{CS})
- net !MREQ: now also U10.19 (~{MREQ}), U6.18 (Q1), U6.19 (Q0), U7.20 (~{CS}), U8.20 (~{CS}), D3.2 (A), D31.2 (A), D5.2 (A), D9.2 (A), U1.12, U1.13, U1.3, U1.4
- net at U12.1 (CA): now also U12.6 (CA), R4.2
- net at U10.17 (~{NMI}): now also R2.2
- net !HALT: now reaches U10.18 (~{HALT})
- net !HALT: now also D24.2 (A)
- net at U10.24 (~{WAIT}): now also R3.2
- net at U10.25 (~{BUSREQ}): now also R1.2
- new net: IC1.3 (X2), Y2.1
- new net: IC1.2 (X1), Y2.2
- new net: BT1.1 (+), IC1.20 (VBAT)
Other:
- note removed: "D0-7 A0-7 TXRX 5VGND IO M1 RD WR ALE RESET INT"
- note removed: "FOR EXTENSION"

Commit message: Add files via upload
Parts:
- U8: value 28C256 -> 28C256 Additional
Connections:
- net !HALT: now also D6.1 (K); no longer D24.2 (A)
- net !INT: now also D9.1 (K); no longer D21.2 (A)
- net !IORQ: now also D18.1 (K); no longer D12.2 (A)
- net !M1: now also D24.1 (K); no longer D6.2 (A)
- net !MREQ: now also D21.1 (K); no longer D9.2 (A)
- net !RD: now also D15.1 (K); no longer D15.2 (A)
- net !RESET: now also SW65.2
- net !WR: now also D12.1 (K); no longer D18.2 (A)
- net 5V: now also D12.2 (A), D15.2 (A), D18.2 (A), D21.2 (A), D24.2 (A), D6.2 (A), D9.2 (A); no longer SW65.1
- net GND: now also SW65.1; no longer D12.1 (K), D15.1 (K), D18.1 (K), D21.1 (K), D24.1 (K), D6.1 (K), D9.1 (K), SW65.2

Commit message: Add files via upload
Parts:
- added J5: Conn_01x40, Connector_PinHeader_2.54mm:PinHeader_1x40_P2.54mm_Vertical, symbol Connector_Generic:Conn_01x40
- added U18, U19: 74AHCT1G32, Package_TO_SOT_SMD:SC-74A-5_1.55x2.9mm_P0.95mm, symbol 74xGxx:74AHCT1G32
Connections:
- net !HALT: now also J5.11 (Pin_11)
- net !INT: now also J5.10 (Pin_10)
- net !IORQ: now also J5.7 (Pin_7)
- net !M1: now also J5.5 (Pin_5)
- net !MREQ: now also J5.6 (Pin_6), U18.2, U19.2; no longer D3.2 (A), D31.2 (A), U1.12, U1.13, U1.3, U10.5 (A_{15}), U2.2 (A), U6.19 (Q0), U7.20 (~{CS}), U9.20 (~{CS})
- net !RD: now also J5.8 (Pin_8)
- net !RESET: now also J5.12 (Pin_12)
- net !WR: now also J5.9 (Pin_9)
- net 5V: now also J5.1 (Pin_1), U18.5 (VCC), U19.5 (VCC)
- net A0: now also J5.16 (Pin_16)
- net A1: now also J5.17 (Pin_17)
- net A10: now also J5.26 (Pin_26)
- net A11: now also J5.27 (Pin_27)
- net A12: now also J5.28 (Pin_28)
- net A13: now also J5.29 (Pin_29)
- net A14: now also J5.30 (Pin_30)
- net A2: now also J5.18 (Pin_18)
- net A3: now also J5.19 (Pin_19)
- net A4: now also J5.20 (Pin_20)
- net A5: now also J5.21 (Pin_21)
- net A6: now also J5.22 (Pin_22)
- net A7: now also J5.23 (Pin_23)
- net A8: now also J5.24 (Pin_24)
- net A9: now also J5.25 (Pin_25)
- net D0: now also J5.33 (Pin_33)
- net D1: now also J5.34 (Pin_34)
- net D2: now also J5.35 (Pin_35)
- net D3: now also J5.36 (Pin_36)
- net D4: now also J5.37 (Pin_37)
- net D5: now also J5.38 (Pin_38)
- net D6: now also J5.39 (Pin_39)
- net D7: now also J5.40 (Pin_40)
- net GND: now also J5.2 (Pin_2), U18.3 (GND), U19.3 (GND)
- net IO1: now also U3.9
- net RX2: now also J5.4 (Pin_4)
- net TX2: now also J5.3 (Pin_3)
- net IO8: now reaches U3.8
- net IO8: now also J5.13 (Pin_13)
- net CLK: now reaches U10.6 (CLK), Y1.8 (OUT)
- net CLK: now also J5.14 (Pin_14)
- new net: U18.4, U9.20 (~{CS})
- new net: U1.12, U19.4, U7.20 (~{CS})
- new net A15: D31.2 (A), J5.31 (Pin_31), U1.13, U1.3, U10.5 (A_{15}), U18.1, U2.2 (A)
- new net BANK_0: D3.2 (A), U19.1, U6.19 (Q0)

Commit message: Add files via upload
Connections:
- net !INT: now also U3.10; no longer U3.11
- net at U16.30 (INTR), U17.30 (INTR): now also U3.11; no longer U3.10
Changed lines of the file:
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@@
 	)
 	(junction
+		(at 158.75 234.95)
+		(diameter 0)
+		(color 0 0 0 0)
+	)
+	(junction
 		(at 375.92 76.2)
 		(diameter 0)
@@
 	)
 	(junction
-		(at 158.75 234.95)
-		(diameter 0)
-		(color 0 0 0 0)
-	)
-	(junction
 		(at 377.19 63.5)
 		(diameter 0)
@@
 	)
 	(symbol
+		(lib_id "74xx:74HC04")
+		(at 151.13 234.95 180)
+		(unit 5)
+		(body_style 1)
+		(exclude_from_sim no)
+		(in_bom yes)
+		(on_board yes)
+		(in_pos_files yes)
+		(dnp no)
+		(fields_autoplaced yes)
+		(property "Reference" "U3"
+			(at 151.13 243.84 0)
+			(hide yes)
+			(show_name no)
+			(do_not_autoplace no)
+			(effects
+				(font
+					(size 1.27 1.27)
+				)
+			)
+		)
+		(property "Value" "74HC04"
+			(at 151.13 228.6 0)
+			(show_name no)
+			(do_not_autoplace no)
+			(effects
+				(font
+					(size 1.27 1.27)
+				)
+			)
+		)
+		(property "Footprint" "Package_DIP:DIP-14_W7.62mm"
+			(at 151.13 234.95 0)
+			(hide yes)
+			(show_name no)
+			(do_not_autoplace no)
+			(effects
+				(font
+					(size 1.27 1.27)
+				)
+			)
+		)
+		(property "Datasheet" "https://assets.nexperia.com/documents/data-sheet/74HC_HCT04.pdf"
+			(at 151.13 234.95 0)
+			(hide yes)
+			(show_name no)
+			(do_not_autoplace no)
+			(effects
+				(font
+					(size 1.27 1.27)
+				)
+			)
+		)
+		(property "Description" "Hex Inverter"
+			(at 151.13 234.95 0)
+			(hide yes)
+			(show_name no)
+			(do_not_autoplace no)
+			(effects
+				(font
+					(size 1.27 1.27)
+				)
+			)
+		)
+		(pin "12"
+		)
+		(pin "14"
+		)
+		(pin "2"
+		)
+		(pin "13"
+		)
+		(pin "3"
+		)
+		(pin "4"
+		)
+		(pin "5"
+		)
+		(pin "9"
+		)
+		(pin "1"
+		)
+		(pin "6"
+		)
+		(pin "10"
+		)
+		(pin "11"
+		)
+		(pin "8"
+		)
+		(pin "7"
+		)
+		(instances
+			(project "z80handheld"
+				(path "/8f7bf91a-544f-4b21-b53f-d26c5f4e4826"
+					(reference "U3")
+					(unit 5)
+				)
+			)
+		)
+	)
+	(symbol
 		(lib_id "Device:LED")
 		(at 267.97 85.09 0)
@@
 				)
 			)
-		)
-	)
-	(symbol
-		(lib_id "74xx:74HC04")
-		(at 151.13 234.95 0)
-		(unit 5)
-		(body_style 1)
-		(exclude_from_sim no)
-		(in_bom yes)
-		(on_board yes)
-		(in_pos_files yes)
-		(dnp no)
-		(fields_autoplaced yes)
-		(property "Reference" "U3"
-			(at 151.13 226.06 0)
-			(hide yes)
-			(show_name no)
-			(do_not_autoplace no)
-			(effects
-				(font
-					(size 1.27 1.27)
-				)
-			)
-		)
-		(property "Value" "74HC04"
-			(at 151.13 228.6 0)
-			(show_name no)
-			(do_not_autoplace no)
-			(effects
-				(font
-					(size 1.27 1.27)
-				)
-			)
-		)
-		(property "Footprint" "Package_DIP:DIP-14_W7.62mm"
-			(at 151.13 234.95 0)
-			(hide yes)
-			(show_name no)
-			(do_not_autoplace no)
-			(effects
-				(font
-					(size 1.27 1.27)
-				)
-			)
-		)
-		(property "Datasheet" "https://assets.nexperia.com/documents/data-sheet/74HC_HCT04.pdf"
-			(at 151.13 234.95 0)
-			(hide yes)
-			(show_name no)
-			(do_not_autoplace no)
-			(effects
-				(font
-					(size 1.27 1.27)
-				)
-			)
-		)
-		(property "Description" "Hex Inverter"
-			(at 151.13 234.95 0)
-			(hide yes)
-			(show_name no)
-			(do_not_autoplace no)
-			(effects
-				(font
-					(size 1.27 1.27)
-				)
-			)
-		)
-		(pin "12"
-		)
-		(pin "14"
-		)
-		(pin "2"
-		)
-		(pin "13"
-		)
-		(pin "3"
-		)
-		(pin "4"
-		)
-		(pin "5"
-		)
-		(pin "9"
-		)
-		(pin "1"
-		)
-		(pin "6"
-		)
-		(pin "10"
-		)
-		(pin "11"
-		)
-		(pin "8"
-		)
-		(pin "7"
-		)
-		(instances
-			(project "z80handheld"
-				(path "/8f7bf91a-544f-4b21-b53f-d26c5f4e4826"
-					(reference "U3")
-					(unit 5)
-				)
-			)

Commit message: Add files via upload
Parts:
- removed U18, U19: 74AHCT1G32, Package_TO_SOT_SMD:SC-74A-5_1.55x2.9mm_P0.95mm, symbol 74xGxx:74AHCT1G32
- added U18: 74HCT00, Package_DIP:DIP-14_W7.62mm, symbol 74xx:74HCT00
Connections:
- net !MREQ: now also U1.3; no longer D5.2 (A), U1.4, U6.18 (Q1), U8.20 (~{CS})
- net 5V: now also U18.14 (VCC)
- net A15: now also U18.1, U18.4; no longer U1.3
- net GND: now also U18.7 (GND)
- net !CS_Main: now reaches U9.20 (~{CS})
- net !CS_Main: now also U18.8
- net at U1.12: now also U18.9; no longer U7.20 (~{CS})
- net BANK_0 renamed !CS_EEPROM
- net !CS_EEPROM: now also U8.20 (~{CS}), U18.3
- new net: U1.4, U18.10, U18.2, U18.5
- new net !CS_RAM: D5.2 (A), U18.6, U6.18 (Q1), U7.20 (~{CS})
Other:
- moved on the sheet: J5

Commit message: Add files via upload
Parts:
- U2: footprint PCM_Package_DIP_AKL:DIP-14_W7.62mm -> Package_DIP:DIP-14_W7.62mm
- U4: footprint PCM_Package_DIP_AKL:DIP-24_W7.62mm -> Package_DIP:DIP-24_W7.62mm
Connections:
- net IO1: no longer IC1.13 (~{CS}), U1.1, U1.5, U1.9, U2.13 (J), U3.1, U3.3, U3.5, U3.9, U4.1 (~{S0}), U4.10 (~{S9}), U4.11 (~{S10}), U4.13 (~{S11}), U4.14 (~{S12}), U4.15 (~{S13}), U4.16 (~{S14}), U4.17 (~{S15}), U4.3 (~{S2}), U4.4 (~{S3}), U4.5 (~{S4}), U4.6 (~{S5}), U4.7 (~{S6}), U4.8 (~{S7}), U4.9 (~{S8})
- net PullIO: now reaches U1.10, U4.19 (~{E1})
- net PullIO: now also U2.13 (J)
- new net: U3.3, U4.6 (~{S5})
- new net: U1.5, U4.3 (~{S2})
- new net: U3.5, U4.7 (~{S6})
- new net: U3.9, U4.9 (~{S8})
- new net: U1.1, U4.1 (~{S0})
- new net: U1.9, U4.4 (~{S3})
- new net: U3.1, U4.5 (~{S4})
- new net IO7: IC1.13 (~{CS}), U4.8 (~{S7})
