File: z80handheld/z80handheld.kicad_sch (KiCad schematic)
At the start: 139 parts, among them IC1 DS12885+, J1 Power, J2 Esp32 C3 Supermini Right, J3 SPI Screen, J4 Esp32 C3 Supermini Left, J5 Conn_01x40, SW1 SW_Push_45deg, SW10 SW_Push_45deg, SW11 SW_Push_45deg, SW12 SW_Push_45deg, SW13 SW_Push_45deg, SW14 SW_Push_45deg, SW15 SW_Push_45deg, SW16 SW_Push_45deg, SW17 SW_Push_45deg, SW18 SW_Push_45deg, SW19 SW_Push_45deg, SW2 SW_Push_45deg, SW20 SW_Push_45deg, SW21 SW_Push_45deg, SW22 SW_Push_45deg, SW23 SW_Push_45deg, SW24 SW_Push_45deg, SW25 SW_Push_45deg, SW26 SW_Push_45deg, SW27 SW_Push_45deg, SW28 SW_Push_45deg, SW29 SW_Push_45deg, SW3 SW_Push_45deg, SW30 SW_Push_45deg, SW31 SW_Push_45deg, SW32 SW_Push_45deg, SW33 SW_Push_45deg, SW34 SW_Push_45deg, SW35 SW_Push_45deg, SW36 SW_Push_45deg, SW37 SW_Push_45deg, SW38 SW_Push_45deg, SW39 SW_Push_45deg, SW4 SW_Push_45deg, SW40 SW_Push_45deg, SW41 SW_Push_45deg, SW42 SW_Push_45deg, SW43 SW_Push_45deg, SW44 SW_Push_45deg, SW45 SW_Push_45deg, SW46 SW_Push_45deg, SW47 SW_Push_45deg, SW48 SW_Push_45deg, SW49 SW_Push_45deg, SW5 SW_Push_45deg, SW50 SW_Push_45deg, SW51 SW_Push_45deg, SW52 SW_Push_45deg, SW53 SW_Push_45deg, SW54 SW_Push_45deg, SW55 SW_Push_45deg, SW56 SW_Push_45deg, SW57 SW_Push_45deg, SW58 SW_Push_45deg, SW59 SW_Push_45deg, SW6 SW_Push_45deg, SW60 SW_Push_45deg, SW61 SW_Push_45deg, SW62 SW_Push_45deg, SW63 SW_Push_45deg, SW64 SW_Push_45deg, SW65 SW_Push, SW7 SW_Push_45deg, SW8 SW_Push_45deg, SW9 SW_Push_45deg, U1 74HC04, U10 Z84C00xxP, U11 74LS573 IO1, U12 HDSP-7501, U13 74LS573, U14 HDSP-7501, U15 74LS573, U16 16550 IO2, U17 16550 IO3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

Commit message: Add files via upload
Parts:
- U12, U14: footprint Display_7Segment:KCSC02-106 -> Display_7Segment:7SegmentLED_LTS6760_LTS6780
Changed lines of the file:
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@@
 			)
 		)
-		(property "Footprint" "Display_7Segment:KCSC02-106"
+		(property "Footprint" "Display_7Segment:7SegmentLED_LTS6760_LTS6780"
 			(at 327.66 266.7 0)
 			(hide yes)
@@
 			)
 		)
-		(property "Footprint" "Display_7Segment:KCSC02-106"
+		(property "Footprint" "Display_7Segment:7SegmentLED_LTS6760_LTS6780"
 			(at 327.66 220.98 0)
 			(hide yes)
